File: qaxe/qaxe.kicad_pcb (KiCad board)
At the start: 4 copper layers, 89 x 134 mm, 225 parts, among them J1 Barrel_Jack_Switch, J2 Conn_01x06, J3 SWD, J4 Conn_01x02, J5 Conn_01x02, J6 USB_C_Receptacle_USB2.0, M1 Fan_4pin, M2 Fan_4pin, Q3 CSD16415Q5T, Q4 CSD16415Q5T, Q5 CSD16415Q5T, Q6 CSD16415Q5T, Q7 BSS138, U19 BM1366_mode1, U20 BM1366_mode1, U25 BM1366_mode1, U26 BM1366_mode1, U29 TXU0101, U3 LTC3856, U32 TMP1075, U33 TMP1075, U35 STM32L151C8TxA, U36 LM1117-3.3, U37 TXU0101, U38 TXU0101, U39 TXU0101, U4 MCP1824T-0802E, U6 AP3211, U7 MCP1824T-1802E, U8 25MHz, X1 8MHz

Commit message: rev3
Parts:
- removed C89, C90: 100µ/6.3V, qaxe:C_1210_3225Metric
- removed NT5, NT6: NetTie_2, qaxe:NetTie-2_SMD_Pad0.5mm
- removed the REF** at (95.0, 121.9)
- removed TP10, TP11, TP12, TP13, TP2, TP3, TP4, TP5, TP6, TP7, TP8, TP9: TestPoint, qaxe:TestPoint_Pad_D1.5mm
- added C106: 4.7µ/6.3V, Capacitor_SMD:C_1206_3216Metric, F.Cu at (107.7, 63.7)
- added SW1: boot, Button_Switch_SMD:SW_Push_1P1T_NO_CK_KMR2, F.Cu at (99.7, 42.3)
- C1, C100, C101, C102, C103, C104, C18, C2, C20, C21, C22, C24, C25, C26, C27, C28, C29, C3, C30, C31, C32, C33, C34, C35, C36, C37, C38, C4, C40, C41, C42, C43, C44, C46, C47, C49, C5, C50, C51, C52, C53, C54, C55, C56, C57, C58, C59, C6, C60, C61, C62, C63, C64, C65, C66, C67, C68, C69, C7, C70, C71, C72, C73, C74, C75, C76, C77, C78, C79, C8, C80, C81, C82, C83, C84, C85, C86, C87, C88, C9, C93, C94, C96, C99: footprint qaxe:C_0805_2012Metric -> Capacitor_SMD:C_0805_2012Metric
- C10, C105, C11, C12, C13, C14, C16, C91, C92: footprint qaxe:C_1210_3225Metric -> Capacitor_SMD:C_1210_3225Metric
- C15, C17: footprint qaxe:C_1210_3225Metric -> Capacitor_SMD:C_1210_3225Metric; moved to B.Cu
- C19, C23, C97, C98: footprint qaxe:C_1206_3216Metric -> Capacitor_SMD:C_1206_3216Metric
- C39, C45, C48: footprint qaxe:CP_EIA-7343-15_Kemet-W -> Capacitor_Tantalum_SMD:CP_EIA-7343-15_Kemet-W; moved to F.Cu
- C95: footprint qaxe:CP_Elec_8x10 -> Capacitor_SMD:CP_Elec_8x10
- D1: footprint qaxe:D_SMB -> Diode_SMD:D_SMB
- D2, D3: footprint qaxe:D_SOD-323 -> Diode_SMD:D_SOD-323
- D4: footprint qaxe:D_SOD-128 -> Diode_SMD:D_SOD-128
- D5, D6: footprint qaxe:LED_1206_3216Metric -> LED_SMD:LED_1206_3216Metric
- F1: footprint qaxe:fuseholder_littlefuse_blok -> myfootprints:fuseholder_littlefuse_blok
- J1: footprint qaxe:BarrelJack_CUI_PJ-102AH_Horizontal -> Connector_BarrelJack:BarrelJack_CUI_PJ-102AH_Horizontal
- J2: footprint qaxe:PinHeader_1x06_P1.27mm_Vertical -> Connector_PinHeader_1.27mm:PinHeader_1x06_P1.27mm_Vertical
- J3: footprint qaxe:PinHeader_IDC_2x05_P1.27mm_Vertical_SMD -> myfootprints:PinHeader_IDC_2x05_P1.27mm_Vertical_SMD
- J4, J5: footprint qaxe:PinHeader_1x02_P2.54mm_Vertical -> Connector_PinHeader_2.54mm:PinHeader_1x02_P2.54mm_Vertical
- J6: footprint qaxe:USB_C_Receptacle_GCT_USB4105-xx-A_16P_TopMnt_Horizontal -> Connector_USB:USB_C_Receptacle_GCT_USB4105-xx-A_16P_TopMnt_Horizontal
- L1, L2: footprint qaxe:IFLR-4031GC-01-8x10 -> myfootprints:IFLR-4031GC-01-8x10
- L3: footprint qaxe:L_Taiyo-Yuden_NR-50xx -> Inductor_SMD:L_Taiyo-Yuden_NR-50xx
- M1, M2: footprint qaxe:FanPinHeader_1x04_P2.54mm_Vertical -> Connector:FanPinHeader_1x04_P2.54mm_Vertical
- NT1, NT2, NT3, NT4: footprint qaxe:NetTie-2_SMD_Pad0.5mm -> NetTie:NetTie-2_SMD_Pad0.5mm
- NT7: footprint qaxe:NetTie-2_L3_SMD_Pad0.5mm -> myfootprints:NetTie-2_L3_SMD_Pad0.5mm
- Q3, Q4, Q5, Q6: footprint qaxe:VSONP-8-1EP_5x6_P1.27mm -> Package_SON:VSONP-8-1EP_5x6_P1.27mm
- Q7: footprint qaxe:SOT-23 -> Package_TO_SOT_SMD:SOT-23
- R1, R10, R11, R14, R15, R16, R17, R19, R2, R20, R21, R22, R23, R24, R25, R26, R27, R28, R29, R30, R31, R32, R34, R35, R36, R37, R38, R39, R4, R40, R42, R5, R6, R7, R8, R9: footprint qaxe:R_0805_2012Metric -> Resistor_SMD:R_0805_2012Metric
- R12, R13: footprint qaxe:R_2010_5025Metric -> Resistor_SMD:R_2010_5025Metric
- R18: footprint qaxe:R_1210_3225Metric -> Resistor_SMD:R_1210_3225Metric
- R3: footprint qaxe:R_1206_3216Metric -> Resistor_SMD:R_1206_3216Metric
- R33, R41: value 2k7 -> 2.7k; footprint qaxe:R_0805_2012Metric -> Resistor_SMD:R_0805_2012Metric
- TP1, TP14, TP15: footprint qaxe:TestPoint_Pad_2.0x2.0mm -> TestPoint:TestPoint_Pad_2.0x2.0mm
- U29, U37, U38, U39: footprint qaxe:SOT-363_SC-70-6 -> Package_TO_SOT_SMD:SOT-363_SC-70-6
- U3: footprint qaxe:QFN-32-1EP_5x5mm_P0.5mm_EP3.45x3.45mm_ThermalVias -> Package_DFN_QFN:QFN-32-1EP_5x5mm_P0.5mm_EP3.45x3.45mm_ThermalVias
- U32, U33: footprint qaxe:TMP1075-DRL -> myfootprints:TMP1075-DRL
- U35: footprint qaxe:LQFP-48_7x7mm_P0.5mm -> Package_QFP:LQFP-48_7x7mm_P0.5mm
- U36: value LM1117-3.3 -> 1117-3.3; footprint qaxe:SOT-223-3_TabPin2 -> Package_TO_SOT_SMD:SOT-223-3_TabPin2
- U4, U7: footprint qaxe:SOT-23-5 -> Package_TO_SOT_SMD:SOT-23-5
- U6: footprint qaxe:SOT-23-6 -> Package_TO_SOT_SMD:SOT-23-6
- U8, X1: footprint qaxe:Oscillator_SMD_EuroQuartz_XO32-4Pin_3.2x2.5mm -> Oscillator:Oscillator_SMD_EuroQuartz_XO32-4Pin_3.2x2.5mm
- moved C48 51.6 mm to (110.9, 68.5), turned to 0 degrees
- moved C15 51.4 mm to (94.9, 119.0), turned to -90 degrees
- moved C45 50.9 mm to (110.9, 78.1), turned to 0 degrees
- moved C17 50.4 mm to (94.9, 125.3), turned to 90 degrees
- moved C39 31.9 mm to (110.9, 73.3)
- moved TP15 21.6 mm to (114.3, 82.6)
- moved TP14 18.0 mm to (103.7, 82.6)
- moved C10 11.4 mm to (110.5, 63.7), turned to 90 degrees
- moved R39 10.9 mm to (111.6, 40.9)
- moved NT7 10.7 mm to (73.4, 48.3), turned to 180 degrees
- moved C12 9.30 mm to (104.0, 68.4), turned to 180 degrees
- moved R30 7.33 mm to (97.5, 46.3)
- moved R41 6.98 mm to (114.4, 41.9), turned to 90 degrees
- moved J5 3.67 mm to (104.5, 41.3), turned to 0 degrees
- moved R14 3.20 mm to (109.9, 71.2)
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Connections:
- R14 pad 1: Net-(NT5-Pad1) -> +1V2
- R15 pad 1: Net-(NT6-Pad1) -> GND
Routing:
- net Net-(U20-ADDR0): track 17.7 -> 0.00 mm, vias 1 -> 0
- net Net-(U35-BOOT0): track 1.78 -> 17.3 mm
- net Net-(U25-ADDR1): track 15.5 -> 0.00 mm, vias 1 -> 0
- net Net-(U26-ADDR0): track 12.1 -> 0.00 mm, vias 1 -> 0
- net Net-(U25-ADDR0): track 11.1 -> 0.00 mm, vias 1 -> 0
- net Net-(U26-ADDR1): track 10.9 -> 0.00 mm, vias 1 -> 0
- net Net-(U20-PIN_MODE): track 8.84 -> 0.00 mm, vias 1 -> 0
- net Net-(U26-PIN_MODE): track 8.18 -> 0.00 mm, vias 1 -> 0
- net Net-(U19-ADDR0): track 8.05 -> 0.00 mm, vias 1 -> 0
- net Net-(U20-ADDR1): track 8.02 -> 0.00 mm, vias 1 -> 0
- net Net-(U19-PIN_MODE): track 7.15 -> 0.00 mm, vias 1 -> 0
- net Net-(U19-ADDR1): track 7.10 -> 0.00 mm, vias 1 -> 0
- net Net-(U25-PIN_MODE): track 6.93 -> 0.00 mm, vias 1 -> 0
- net GND: track 261.7 -> 267.0 mm, vias 223 -> 228
- net /STM32/TACHO2: track 38.3 -> 33.7 mm
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Other:
- board text added: "V0.3"
- board text removed: "V0.02"

Commit message: updated ibom
Parts:
- R6: value 20k -> 22k
Changed lines of the file:
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@@
         (effects (font (size 0.8 0.8) (thickness 0.15)))
     )
-    (fp_text value "20k" (at 0 1.65 90) (layer "F.Fab")
+    (fp_text value "22k" (at 0 1.65 90) (layer "F.Fab")
         (effects (font (size 1 1) (thickness 0.15)))
     )
@@
       (net 8 "Net-(U3-SENSE1-)") (pinfunction "SENSE1-") (pintype "input"))
     (pad "33" thru_hole circle (at -1 -1 270) (size 0.5 0.5) (drill 0.3) (layers "*.Cu")
-      (net 1 "GND") (pinfunction "SGND") (pintype "power_in"))
+      (net 1 "GND") (pinfunction "PGND") (pintype "power_in"))
     (pad "33" thru_hole circle (at -1 0 270) (size 0.5 0.5) (drill 0.3) (layers "*.Cu")
-      (net 1 "GND") (pinfunction "SGND") (pintype "power_in"))
+      (net 1 "GND") (pinfunction "PGND") (pintype "power_in"))
     (pad "33" thru_hole circle (at -1 1 270) (size 0.5 0.5) (drill 0.3) (layers "*.Cu")
-      (net 1 "GND") (pinfunction "SGND") (pintype "power_in"))
+      (net 1 "GND") (pinfunction "PGND") (pintype "power_in"))
     (pad "33" thru_hole circle (at 0 -1 270) (size 0.5 0.5) (drill 0.3) (layers "*.Cu")
-      (net 1 "GND") (pinfunction "SGND") (pintype "power_in"))
+      (net 1 "GND") (pinfunction "PGND") (pintype "power_in"))
     (pad "33" thru_hole circle (at 0 0 270) (size 0.5 0.5) (drill 0.3) (layers "*.Cu")
-      (net 1 "GND") (pinfunction "SGND") (pintype "power_in"))
+      (net 1 "GND") (pinfunction "PGND") (pintype "power_in"))
     (pad "33" smd rect (at 0 0 270) (size 2.5 2.5) (layers "B.Cu")
-      (net 1 "GND") (pinfunction "SGND") (pintype "power_in"))
+      (net 1 "GND") (pinfunction "PGND") (pintype "power_in"))
     (pad "33" smd rect (at 0 0 270) (size 3.45 3.45) (layers "F.Cu" "F.Mask")
-      (net 1 "GND") (pinfunction "SGND") (pintype "power_in"))
+      (net 1 "GND") (pinfunction "PGND") (pintype "power_in"))
     (pad "33" thru_hole circle (at 0 1 270) (size 0.5 0.5) (drill 0.3) (layers "*.Cu")
-      (net 1 "GND") (pinfunction "SGND") (pintype "power_in"))
+      (net 1 "GND") (pinfunction "PGND") (pintype "power_in"))
     (pad "33" thru_hole circle (at 1 -1 270) (size 0.5 0.5) (drill 0.3) (layers "*.Cu")
-      (net 1 "GND") (pinfunction "SGND") (pintype "power_in"))
+      (net 1 "GND") (pinfunction "PGND") (pintype "power_in"))
     (pad "33" thru_hole circle (at 1 0 270) (size 0.5 0.5) (drill 0.3) (layers "*.Cu")
-      (net 1 "GND") (pinfunction "SGND") (pintype "power_in"))
+      (net 1 "GND") (pinfunction "PGND") (pintype "power_in"))
     (pad "33" thru_hole circle (at 1 1 270) (size 0.5 0.5) (drill 0.3) (layers "*.Cu")
-      (net 1 "GND") (pinfunction "SGND") (pintype "power_in"))
+      (net 1 "GND") (pinfunction "PGND") (pintype "power_in"))
     (model "${KICAD6_3DMODEL_DIR}/Package_DFN_QFN.3dshapes/QFN-32-1EP_5x5mm_P0.5mm_EP3.45x3.45mm.wrl"
       (offset (xyz 0 0 0))
@@
     (descr "CK components KMR2 tactile switch http://www.ckswitches.com/media/1479/kmr2.pdf")
     (tags "tactile switch kmr2")
+    (property "Distributor" "D")
+    (property "Manufacturer" "KMR221GLFS")
+    (property "OrderNr" "401-1427-1-ND")
     (property "Sheetfile" "pi.kicad_sch")
     (property "Sheetname" "STM32")
