File: qaxe/qaxe.kicad_pcb (KiCad board)
At the start: 4 copper layers, 89 x 134 mm, 210 parts, among them J1 Barrel_Jack_Switch, J2 Conn_01x06, J3 SWD, J4 Conn_01x02, J5 Conn_01x02, J6 USB_C_Receptacle_USB2.0, M1 Fan_4pin, M2 Fan_4pin, Q3 CSD16415Q5T, Q4 CSD16415Q5T, Q5 CSD16415Q5T, Q6 CSD16415Q5T, Q7 BSS138, SW1 boot, U19 BM1366_mode1, U20 BM1366_mode1, U25 BM1366_mode1, U26 BM1366_mode1, U29 TXU0101, U3 LTC3856, U32 TMP1075, U33 TMP1075, U35 STM32L151C8TxA, U36 1117-3.3, U37 TXU0101, U38 TXU0101, U39 TXU0101, U4 MCP1824T-0802E, U6 AP3211, U7 MCP1824T-1802E, U8 25MHz, X1 8MHz

Commit message: updated board with -CC variant
Parts:
- U35: value STM32L151C8TxA -> STM32L151CCT6
Changed lines of the file:
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@@
     (tags "LQFP QFP")
     (property "Distributor" "D")
-    (property "Manufacturer" "STM32L151C8T6A")
-    (property "OrderNr" "497-17514-ND")
+    (property "Manufacturer" "STM32L151CCT6")
+    (property "OrderNr" "497-19371-1-ND")
     (property "Sheetfile" "pi.kicad_sch")
     (property "Sheetname" "STM32")
@@
         (effects (font (size 0.8 0.8) (thickness 0.15)))
     )
-    (fp_text value "STM32L151C8TxA" (at 0 5.85) (layer "F.Fab")
+    (fp_text value "STM32L151CCT6" (at 0 5.85) (layer "F.Fab")
         (effects (font (size 1 1) (thickness 0.15)))
     )

Commit message: v0.31
Parts:
- added R43: 10k, Resistor_SMD:R_0805_2012Metric, F.Cu at (101.7, 58.9)
- moved R33 0.09 mm to (104.3, 58.3)
Connections:
- U35 pad 20: unconnected-(U35-PB2-Pad20) -> Net-(U35-PB2)
Routing:
- net Net-(U35-PB2): track 0.00 -> 6.77 mm
- net /STM32/LED2: track 13.7 -> 8.00 mm
- net /STM32/LED1: track 9.65 -> 7.68 mm
- net GND: track 267.0 -> 267.8 mm, vias 228 -> 229
Other:
- board text added: "V0.31"
- board text removed: "V0.3"

Commit message: rev3.2
Parts:
- moved C17 3.00 mm to (94.9, 128.3)
- moved C63 3.00 mm to (99.3, 128.6)
- moved C15 3.00 mm to (94.9, 122.0)
- moved C25 3.00 mm to (83.0, 108.1)
- moved C26 3.00 mm to (89.0, 119.3)
- moved C27 3.00 mm to (89.0, 135.3)
- moved C28 3.00 mm to (85.1, 111.6)
- moved C29 3.00 mm to (100.9, 118.7)
- moved C30 3.00 mm to (84.2, 122.1)
- moved C31 3.00 mm to (100.9, 134.6)
- moved C32 3.00 mm to (84.9, 138.9)
- moved C33 3.00 mm to (89.0, 115.3)
- moved C34 3.00 mm to (104.9, 111.7)
- moved C35 3.00 mm to (89.1, 111.5)
- moved C36 3.00 mm to (100.9, 138.9)
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Routing:
- net /STM32/SDA2: track 118.3 -> 121.3 mm
- net /STM32/SCL2: track 117.1 -> 120.1 mm
- net /STM32/ALERT2: track 113.8 -> 116.8 mm
- net +3V3: track 178.9 -> 181.9 mm
- net +0V8: track 173.2 -> 174.7 mm
- net +1V8: track 218.2 -> 219.5 mm
- net /BM1366/RST_N: track 76.4 -> 77.7 mm
- net /BM1366/RO: track 73.6 -> 74.8 mm
- net /BM1366/CI: track 74.4 -> 75.7 mm
Other:
- board size 89 x 134 mm -> 89 x 137 mm
- board text added: "V0.32"
- board text removed: "V0.31"
