File: qaxe/qaxe.kicad_pcb (KiCad board)
At the start: 4 copper layers, 89 x 137 mm, 211 parts, among them J1 Barrel_Jack_Switch, J2 Conn_01x06, J3 SWD, J4 Conn_01x02, J5 Conn_01x02, J6 USB_C_Receptacle_USB2.0, M1 Fan_4pin, M2 Fan_4pin, Q3 CSD16415Q5T, Q4 CSD16415Q5T, Q5 CSD16415Q5T, Q6 CSD16415Q5T, Q7 BSS138, SW1 boot, U19 BM1366_mode1, U20 BM1366_mode1, U25 BM1366_mode1, U26 BM1366_mode1, U29 TXU0101, U3 LTC3856, U32 TMP1075, U33 TMP1075, U35 STM32L151CCT6, U36 1117-3.3, U37 TXU0101, U38 TXU0101, U39 TXU0101, U4 MCP1824T-0802E, U6 AP3211, U7 MCP1824T-1802E, U8 25MHz, X1 8MHz

Commit message: 1368 support
Parts:
- U19, U20, U25, U26: footprint qaxe:BM1366 -> myfootprints:BM1368-smaller
- moved U19 0.25 mm to (87.8, 117.5)
- moved U20 0.25 mm to (102.2, 132.5)
- moved U25 0.25 mm to (87.8, 132.5)
- moved U26 0.25 mm to (102.2, 117.5)
Connections:
- C62 pad 2: Net-(U19-VDD1_1) -> Net-(U19-VDD3_1)
- C63 pad 2: Net-(U20-VDD1_1) -> Net-(U20-VDD3_1)
- C66 pad 1: Net-(U19-VDD1_1) -> Net-(U19-VDD3_1)
- C67 pad 1: Net-(U20-VDD1_1) -> Net-(U20-VDD3_1)
- C69 pad 2: Net-(U19-VDD3_1) -> Net-(U19-VDD1_1)
- C70 pad 2: Net-(U20-VDD3_1) -> Net-(U20-VDD1_1)
- C71 pad 1: Net-(U19-VDD3_1) -> Net-(U19-VDD1_1)
- C72 pad 1: Net-(U20-VDD3_1) -> Net-(U20-VDD1_1)
- C73 pad 2: Net-(U25-VDD1_1) -> Net-(U25-VDD3_1)
- C74 pad 2: Net-(U26-VDD1_1) -> Net-(U26-VDD3_1)
- C75 pad 1: Net-(U25-VDD1_1) -> Net-(U25-VDD3_1)
- C76 pad 1: Net-(U26-VDD1_1) -> Net-(U26-VDD3_1)
- C77 pad 2: Net-(U25-VDD3_1) -> Net-(U25-VDD1_1)
- C78 pad 2: Net-(U26-VDD3_1) -> Net-(U26-VDD1_1)
- C79 pad 1: Net-(U25-VDD3_1) -> Net-(U25-VDD1_1)
- C80 pad 1: Net-(U26-VDD3_1) -> Net-(U26-VDD1_1)
- C93 pad 1: Net-(U19-VDD1_1) -> Net-(U19-VDD3_1)
- C94 pad 1: Net-(U20-VDD1_1) -> Net-(U20-VDD3_1)
- J6 pad A4: unconnected-(J6-VBUS-PadA4) -> /STM32/X
- J6 pad A9: unconnected-(J6-VBUS-PadA4) -> /STM32/X
- J6 pad B4: unconnected-(J6-VBUS-PadA4) -> /STM32/X
- J6 pad B9: unconnected-(J6-VBUS-PadA4) -> /STM32/X
- U19 pad 10: Net-(U19-ADDR0) -> unconnected-(U19-?-Pad10)
- U19 pad 11: Net-(U19-ADDR1) -> unconnected-(U19-?-Pad11)
- U19 pad 12: GND -> unconnected-(U19-?-Pad12)
- U19 pad 13: +0V8 -> GND
- U19 pad 14: +1V8 -> +0V8
- U19 pad 16: +0V8 -> +1V8
- U19 pad 17: GND -> +0V8
- U19 pad 18: Net-(U19-PIN_MODE) -> GND
- U19 pad 20: Net-(U19-CO) -> unconnected-(U19-?-Pad20)
- U19 pad 21: Net-(U19-CLKO) -> unconnected-(U19-?-Pad21)
- U19 pad 22: Net-(U19-RI) -> Net-(U19-BO)
- U19 pad 23: Net-(U19-BO) -> Net-(U19-CO)
- U19 pad 24: Net-(U19-NRSTO) -> Net-(U19-RI)
- U19 pad 25: GND -> Net-(U19-CLKO)
- U19 pad 26: Net-(U19-VDD3_1) -> Net-(U19-NRSTO)
- U19 pad 27: Net-(U19-VDD2_1) -> GND
- U19 pad 29: +1V2 -> Net-(U19-VDD2_1)
- U19 pad 30: GND -> Net-(U19-VDD3_1)
- U19 pad 6: /BM1366/BI -> /BM1366/CI
- U19 pad 9: /BM1366/CI -> /BM1366/BI
- U20 pad 10: Net-(U20-ADDR0) -> unconnected-(U20-?-Pad10)
- U20 pad 11: Net-(U20-ADDR1) -> unconnected-(U20-?-Pad11)
- U20 pad 12: GND -> unconnected-(U20-?-Pad12)
- U20 pad 13: +0V8 -> GND
- U20 pad 14: +1V8 -> +0V8
- U20 pad 16: +0V8 -> +1V8
- U20 pad 17: GND -> +0V8
- U20 pad 18: Net-(U20-PIN_MODE) -> GND
- U20 pad 20: Net-(U20-CO) -> unconnected-(U20-?-Pad20)
- U20 pad 21: Net-(U20-CLKO) -> unconnected-(U20-?-Pad21)
- U20 pad 22: Net-(U20-RI) -> Net-(U20-BO)
- U20 pad 23: Net-(U20-BO) -> Net-(U20-CO)
- U20 pad 24: Net-(U20-NRSTO) -> Net-(U20-RI)
- U20 pad 25: GND -> Net-(U20-CLKO)
- U20 pad 26: Net-(U20-VDD3_1) -> Net-(U20-NRSTO)
- U20 pad 27: Net-(U20-VDD2_1) -> GND
- U20 pad 29: +1V2 -> Net-(U20-VDD2_1)
- U20 pad 30: GND -> Net-(U20-VDD3_1)
- U20 pad 6: Net-(U20-BI) -> Net-(U20-CI)
- U20 pad 9: Net-(U20-CI) -> Net-(U20-BI)
- U25 pad 1: Net-(U19-VDD1_1) -> Net-(U19-VDD3_1)
- U25 pad 10: Net-(U25-ADDR0) -> unconnected-(U25-?-Pad10)
- U25 pad 11: Net-(U25-ADDR1) -> unconnected-(U25-?-Pad11)
- U25 pad 12: GND -> unconnected-(U25-?-Pad12)
- U25 pad 13: +0V8 -> GND
- U25 pad 14: +1V8 -> +0V8
- U25 pad 16: +0V8 -> +1V8
- U25 pad 17: GND -> +0V8
- U25 pad 18: Net-(U25-PIN_MODE) -> GND
- U25 pad 20: Net-(U20-CI) -> unconnected-(U25-?-Pad20)
- U25 pad 21: Net-(U20-CLKI) -> unconnected-(U25-?-Pad21)
- U25 pad 22: Net-(U20-RO) -> Net-(U20-BI)
- U25 pad 23: Net-(U20-BI) -> Net-(U20-CLKI)
- U25 pad 24: Net-(U20-NRSTI) -> Net-(U20-RO)
- U25 pad 25: GND -> Net-(U20-CI)
- U25 pad 26: Net-(U25-VDD3_1) -> Net-(U20-NRSTI)
- U25 pad 27: Net-(U25-VDD2_1) -> GND
- U25 pad 29: +1V2 -> Net-(U25-VDD2_1)
- U25 pad 3: Net-(U19-VDD3_1) -> Net-(U19-VDD1_1)
- U25 pad 30: GND -> Net-(U25-VDD3_1)
- U25 pad 6: Net-(U19-BO) -> Net-(U19-CLKO)
- U25 pad 8: Net-(U19-CLKO) -> Net-(U19-CO)
- U25 pad 9: Net-(U19-CO) -> Net-(U19-BO)
- U26 pad 1: Net-(U20-VDD1_1) -> Net-(U20-VDD3_1)
- U26 pad 10: Net-(U26-ADDR0) -> unconnected-(U26-?-Pad10)
- U26 pad 11: Net-(U26-ADDR1) -> unconnected-(U26-?-Pad11)
- U26 pad 12: GND -> unconnected-(U26-?-Pad12)
- U26 pad 13: +0V8 -> GND
- U26 pad 14: +1V8 -> +0V8
- U26 pad 16: +0V8 -> +1V8
- U26 pad 17: GND -> +0V8
- U26 pad 18: Net-(U26-PIN_MODE) -> GND
- U26 pad 22: Net-(U26-RI) -> unconnected-(U26-BO-Pad22)
- U26 pad 24: unconnected-(U26-NRSTO-Pad24) -> Net-(U26-RI)
- U26 pad 25: GND -> unconnected-(U26-CLKO-Pad25)
- U26 pad 26: Net-(U26-VDD3_1) -> unconnected-(U26-NRSTO-Pad26)
- U26 pad 27: Net-(U26-VDD2_1) -> GND
- U26 pad 29: +1V2 -> Net-(U26-VDD2_1)
- U26 pad 3: Net-(U20-VDD3_1) -> Net-(U20-VDD1_1)
- U26 pad 30: GND -> Net-(U26-VDD3_1)
- U26 pad 6: Net-(U20-BO) -> Net-(U20-CLKO)
- U26 pad 8: Net-(U20-CLKO) -> Net-(U20-CO)
- U26 pad 9: Net-(U20-CO) -> Net-(U20-BO)
Routing:
- net Net-(U20-CI): track 23.6 -> 16.7 mm
- net unconnected-(J6-VBUS-PadA4): track 6.55 -> 0.00 mm
- net /STM32/X: track 0.00 -> 6.55 mm
- net Net-(U20-BI): track 17.1 -> 23.6 mm
- net +0V8: track 174.7 -> 168.2 mm
- net Net-(U19-VDD3_1): track 11.6 -> 15.1 mm, vias 1 -> 2
- net Net-(U19-VDD1_1): track 15.1 -> 11.6 mm, vias 2 -> 1
- net Net-(U25-VDD3_1): track 6.37 -> 3.95 mm
- net Net-(U25-VDD1_1): track 3.95 -> 6.37 mm
- net Net-(U20-VDD3_1): track 12.7 -> 14.9 mm, vias 1 -> 2
- net Net-(U20-VDD1_1): track 14.9 -> 12.7 mm, vias 2 -> 1
- net /BM1366/CI: track 75.7 -> 73.5 mm
- net +1V8: track 219.5 -> 221.3 mm
- net GND: track 267.8 -> 269.1 mm, vias 229 -> 251
- net Net-(U26-VDD3_1): track 6.85 -> 5.61 mm
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Other:
- board text added: "+"
- board text added: "rev4"
- board text removed: "V0.32"

Commit message: gerbers for 1368
Parts:
- U19, U20, U25, U26: value BM1366_mode1 -> BM1368_mode1
Changed lines of the file:
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@@
 			)
 		)
-		(property "Value" "BM1366_mode1"
+		(property "Value" "BM1368_mode1"
 			(at 0.07 5.189 -90)
 			(unlocked yes)
@@
 			)
 		)
-		(property "Value" "BM1366_mode1"
+		(property "Value" "BM1368_mode1"
 			(at 0.07 5.189 -90)
 			(unlocked yes)
@@
 			)
 		)
-		(property "Value" "BM1366_mode1"
+		(property "Value" "BM1368_mode1"
 			(at 0.07 5.189 90)
 			(unlocked yes)
@@
 			)
 		)
-		(property "Value" "BM1366_mode1"
+		(property "Value" "BM1368_mode1"
 			(at 0.07 5.189 90)
 			(unlocked yes)
