File: qaxe/power.kicad_sch (KiCad schematic)
At the start: 74 parts, among them Q3 CSD16415Q5T, Q4 CSD16415Q5T, Q7 CSD16415Q5T, Q8 CSD16415Q5T, U17 LTC3856, U3 AP3211, U36 1117-3.3, U4 +0V8, U5 MCP1824T-1802E, U6 MCP1824T-0802E

Commit message: fixed wrong lm1117 variant in bom
Parts:
- U36: Manufacturer LM1117IMPX-ADJNOPB -> LM1117IMPX-3.3/NOPB; OrderNr 488-LM1117IMPX-ADJNOPBCT-ND -> LM1117IMPX-3.3/NOPBCT-ND
Changed lines of the file:
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@@
       (effects (font (size 1.27 1.27)) hide)
     )
-    (property "Manufacturer" "LM1117IMPX-ADJNOPB" (at 378.46 166.37 0)
+    (property "Manufacturer" "LM1117IMPX-3.3/NOPB" (at 378.46 166.37 0)
       (effects (font (size 1.27 1.27)) hide)
     )
-    (property "OrderNr" "488-LM1117IMPX-ADJNOPBCT-ND" (at 378.46 166.37 0)
+    (property "OrderNr" "LM1117IMPX-3.3/NOPBCT-ND" (at 378.46 166.37 0)
       (effects (font (size 1.27 1.27)) hide)
     )

Commit message: 1368 support
Parts:
- renumbered C23 to C18, C25 to C20, U4 to U2, U6 to U4, U4 to U5, U5 to U7
