File: qaxe/bm1366.kicad_sch (KiCad schematic)
At the start: 108 parts, among them J2 Conn_01x06, Q7 BSS138, U10 +0V8, U11 +0V8, U12 +0V8, U13 +0V8, U14 +0V8, U15 +0V8, U16 +0V8, U17 +0V8, U18 +0V8, U19 BM1366_mode1, U20 BM1366_mode1, U21 +0V8, U22 +0V8, U23 +0V8, U24 +0V8, U25 BM1366_mode1, U26 BM1366_mode1, U27 +0V8, U28 +0V8, U29 TXU0101, U31 +0V8, U34 +0V8, U38 TXU0101, U8 25MHz, U9 +0V8

Commit message: updated BOM and replaces bss138 and 3.3V LDO with parts that are available
Parts:
- Q7: Distributor (none) -> D; Manufacturer (none) -> BSS138; OrderNr (none) -> 4530-BSS138CT-ND
Changed lines of the file:
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@@
       (effects (font (size 1.27 1.27)) (justify left) hide)
+    )
+    (property "Distributor" "D" (at 349.885 108.585 0)
+      (effects (font (size 1.27 1.27)) hide)
+    )
+    (property "Manufacturer" "BSS138" (at 349.885 108.585 0)
+      (effects (font (size 1.27 1.27)) hide)
+    )
+    (property "OrderNr" "4530-BSS138CT-ND" (at 349.885 108.585 0)
+      (effects (font (size 1.27 1.27)) hide)
     )
     (pin "1")

Commit message: rev3
Parts:
- removed C39, C45, C48: 330µ/6.3V, Capacitor_Tantalum_SMD:CP_EIA-7343-15_Kemet-W, symbol Device:C_Polarized
- removed TP10, TP11, TP12, TP13, TP2, TP3, TP4, TP5, TP6, TP7, TP8, TP9: TestPoint, TestPoint:TestPoint_Pad_D1.5mm, symbol Connector:TestPoint
- added C55, C56: 100µ/6.3V, Capacitor_SMD:C_1210_3225Metric, symbol Device:C
Connections:
- net +1V2: now also C55.1, C56.1
- net GND: now also C55.2, C56.2
- no-connect marks 8 -> 20

Commit message: 1368 support
Parts:
- R20, R21, R23: now fitted
- U19, U20, U25, U26: footprint bitaxe:BM1366 -> myfootprints:BM1368-smaller; symbol bitaxe:BM1366_mode1 -> mylib7:BM1368_mode1
Connections:
- net +0V8: now also U19.14 (VDDIO_08_0), U19.17 (VDDIO_08_1), U20.14 (VDDIO_08_0), U20.17 (VDDIO_08_1), U25.14 (VDDIO_08_0), U25.17 (VDDIO_08_1), U26.14 (VDDIO_08_0), U26.17 (VDDIO_08_1); no longer U19.13 (VDDIO_08_0), U19.16 (VDDIO_08_1), U20.13 (VDDIO_08_0), U20.16 (VDDIO_08_1), U25.13 (VDDIO_08_0), U25.16 (VDDIO_08_1), U26.13 (VDDIO_08_0), U26.16 (VDDIO_08_1)
- net +1V2: now also U19.31 (VDD), U20.31 (VDD), U25.31 (VDD), U26.31 (VDD); no longer U19.29 (VDD), U20.29 (VDD), U25.29 (VDD), U26.29 (VDD)
- net +1V8: now also U19.16 (VDDIO_12_1), U20.16 (VDDIO_12_1), U25.16 (VDDIO_12_1), U26.16 (VDDIO_12_1); no longer U19.14 (VDDIO_18_0), U20.14 (VDDIO_18_0), U25.14 (VDDIO_18_0), U26.14 (VDDIO_18_0)
- net BI: now also U19.9 (BI); no longer U19.6 (BI)
- net CI: now also U19.6 (CI); no longer U19.9 (CI)
- net GND: now also U19.13 (PLL_VSS), U19.18 (VSS), U19.27 (VSS), U19.32 (VSS), U20.13 (PLL_VSS), U20.18 (VSS), U20.27 (VSS), U20.32 (VSS), U25.13 (PLL_VSS), U25.18 (VSS), U25.27 (VSS), U25.32 (VSS), U26.13 (PLL_VSS), U26.18 (VSS), U26.27 (VSS), U26.32 (VSS); no longer U19.12 (PLL_VSS), U19.17 (VSS), U19.25 (VDD4_0), U19.30 (GND), U20.12 (PLL_VSS), U20.17 (VSS), U20.25 (VDD4_0), U20.30 (GND), U25.12 (PLL_VSS), U25.17 (VSS), U25.25 (VDD4_0), U25.30 (GND), U26.12 (PLL_VSS), U26.17 (VSS), U26.25 (VDD4_0), U26.30 (GND)
- net at C67.2, C70.1, U26.2 (VDD2_0): now also U20.29 (VDD2_1); no longer U20.27 (VDD2_1)
- net at C70.2, C72.1, U26.3 (VDD1_0): now also U20.28 (VDD1_1); no longer U20.26 (VDD3_1)
- net at R20.1, U25.7 (RO): now also U19.24 (RI); no longer U19.22 (RI)
- net at C69.2, C71.1, U25.3 (VDD1_0): now also U19.28 (VDD1_1); no longer U19.26 (VDD3_1)
- net at C66.2, C69.1, U25.2 (VDD2_0): now also U19.29 (VDD2_1); no longer U19.27 (VDD2_1)
- net at C74.2, C76.1: now also U26.30 (VDD3_1); no longer U26.28 (VDD1_1)
- net at C76.2, C78.1: now also U26.29 (VDD2_1); no longer U26.27 (VDD2_1)
- net at R21.1, U26.7 (RO): now also U20.24 (RI); no longer U20.22 (RI)
- net at C63.2, C67.1, C94.1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: now also U20.30 (VDD3_1); no longer U20.28 (VDD1_1)
- net at C73.2, C75.1: now also U25.30 (VDD3_1); no longer U25.28 (VDD1_1)
- net at C62.2, C66.1, C93.1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: now also U19.30 (VDD3_1); no longer U19.28 (VDD1_1)
- net at U25.20 (?): no longer U20.9 (CI)
- net at U25.21 (?): no longer U20.8 (CLKI)
- net at R23.1, U20.7 (RO): now also U25.24 (RI); no longer U25.22 (RI)
- net at U25.23 (CO): now also U20.8 (CLKI); no longer U20.6 (BI)
- net at U20.5 (NRSTI): now also U25.26 (NRSTO); no longer U25.24 (NRSTO)
- net at C77.2, C79.1: now also U25.28 (VDD1_1); no longer U25.26 (VDD3_1)
- net at C75.2, C77.1: now also U25.29 (VDD2_1); no longer U25.27 (VDD2_1)
- net at U25.5 (NRSTI): now also U19.26 (NRSTO); no longer U19.24 (NRSTO)
- net at U25.6 (CI): now also U19.25 (CLKO); no longer U19.23 (BO)
- net at U25.8 (CLKI): now also U19.23 (CO); no longer U19.21 (CLKO)
- net at U25.9 (BI): now also U19.22 (BO); no longer U19.20 (CO)
- net at C78.2, C80.1: now also U26.28 (VDD1_1); no longer U26.26 (VDD3_1)
- net at R22.1: now also U26.24 (RI); no longer U26.22 (RI)
- net at U26.5 (NRSTI): now also U20.26 (NRSTO); no longer U20.24 (NRSTO)
- net at U26.6 (CI): now also U20.25 (CLKO); no longer U20.23 (BO)
- net at U26.8 (CLKI): now also U20.23 (CO); no longer U20.21 (CLKO)
- net at U26.9 (BI): now also U20.22 (BO); no longer U20.20 (CO)
- new net: U20.9 (BI), U25.22 (BO)
- new net: U20.6 (CI), U25.25 (CLKO)
- no-connect marks 20 -> 28
Other:
- moved on the sheet: C25, C26, C27, C29, C30, C31, C33, C34, C35, C36, C37, C38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

Commit message: gerbers for 1368
Parts:
- U19, U20, U25, U26: value BM1366_mode1 -> BM1368_mode1
Changed lines of the file:
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@@
 			)
 		)
-		(property "Value" "BM1366_mode1"
+		(property "Value" "BM1368_mode1"
 			(at 219.3641 45.72 0)
 			(effects
@@
 			)
 		)
-		(property "Value" "BM1366_mode1"
+		(property "Value" "BM1368_mode1"
 			(at 219.3641 130.81 0)
 			(effects
@@
 			)
 		)
-		(property "Value" "BM1366_mode1"
+		(property "Value" "BM1368_mode1"
 			(at 138.0841 45.72 0)
 			(effects
@@
 			)
 		)
-		(property "Value" "BM1366_mode1"
+		(property "Value" "BM1368_mode1"
 			(at 138.0841 130.81 0)
 			(effects
