File: qaxe/qaxe/qaxe.kicad_pcb (KiCad board)
At the start: 4 copper layers, 89 x 137 mm, 211 parts, among them J1 Barrel_Jack_Switch, J2 Conn_01x06, J3 SWD, J4 Conn_01x02, J5 Conn_01x02, J6 USB_C_Receptacle_USB2.0, M1 Fan_4pin, M2 Fan_4pin, Q3 CSD16415Q5T, Q4 CSD16415Q5T, Q5 CSD16415Q5T, Q6 CSD16415Q5T, Q7 BSS138, SW1 boot, U19 BM1366_mode1, U20 BM1366_mode1, U25 BM1366_mode1, U26 BM1366_mode1, U29 TXU0101, U3 LTC3856, U32 TMP1075, U33 TMP1075, U35 STM32L151CCT6, U36 1117-3.3, U37 TXU0101, U38 TXU0101, U39 TXU0101, U4 MCP1824T-0802E, U6 AP3211, U7 MCP1824T-1802E, U8 25MHz, X1 8MHz

Commit message: updated stm32 to L072 on normal qaxe
Parts:
- U35: value STM32L151CCT6 -> STM32L072CBT6
Connections:
- J6 pad A4: unconnected-(J6-VBUS-PadA4) -> unconnected-(J6-VBUS-PadA4)_2
- J6 pad B4: unconnected-(J6-VBUS-PadA4) -> unconnected-(J6-VBUS-PadA4)_1
- J6 pad B9: unconnected-(J6-VBUS-PadA4) -> unconnected-(J6-VBUS-PadA4)_0
