File: qaxe+/qaxe/qaxe.kicad_pcb (KiCad board)
At the start: 4 copper layers, 89 x 137 mm, 211 parts, among them J1 Barrel_Jack_Switch, J2 Conn_01x06, J3 SWD, J4 Conn_01x02, J5 Conn_01x02, J6 USB_C_Receptacle_USB2.0, M1 Fan_4pin, M2 Fan_4pin, Q3 CSD16415Q5T, Q4 CSD16415Q5T, Q5 CSD16415Q5T, Q6 CSD16415Q5T, Q7 BSS138, SW1 boot, U19 BM1368_mode1, U20 BM1368_mode1, U25 BM1368_mode1, U26 BM1368_mode1, U29 TXU0101, U3 LTC3856, U32 TMP1075, U33 TMP1075, U35 STM32L151CCT6, U36 1117-3.3, U37 TXU0101, U38 TXU0101, U39 TXU0101, U4 MCP1824T-0802E, U6 AP3211, U7 MCP1824T-1802E, U8 25MHz, X1 8MHz

Commit message: updated qaxe+ to L072
Parts:
- U35: value STM32L151CCT6 -> STM32L072CBT6
Changed lines of the file:
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@@
 			)
 		)
-		(property "Value" "STM32L151CCT6"
+		(property "Value" "STM32L072CBT6"
 			(at 0 5.85 0)
 			(layer "F.Fab")
@@
 			)
 		)
-		(property "Manufacturer" "STM32L151CCT6"
+		(property "Manufacturer" "STM32L072CBT6"
 			(at 0 0 0)
 			(layer "F.Fab")
@@
 			)
 		)
-		(property "OrderNr" "497-19371-1-ND"
+		(property "OrderNr" "497-17503-ND"
 			(at 0 0 0)
 			(layer "F.Fab")

Commit message: qaxe+
Parts:
- added JP1: SolderJumper_2_Open, Jumper:SolderJumper-2_P1.3mm_Open_RoundedPad1.0x1.5mm, F.Cu at (54.4, 49.2)
- added JP2: SolderJumper_2_Open, Jumper:SolderJumper-2_P1.3mm_Open_RoundedPad1.0x1.5mm, F.Cu at (92.6, 52.6)
- added R44: 1k, Resistor_SMD:R_0805_2012Metric, B.Cu at (102.8, 138.9)
- added R45: 1k, Resistor_SMD:R_0805_2012Metric, B.Cu at (103.0, 121.5)
- added R46: 1k, Resistor_SMD:R_0805_2012Metric, B.Cu at (85.3, 114.7)
- added R47: 1k, Resistor_SMD:R_0805_2012Metric, B.Cu at (86.9, 128.6)
- added R48: 10k, Resistor_SMD:R_0805_2012Metric, F.Cu at (138.9, 64.8)
- added REF**: stencil-registration, myfootprints:stencil-registration, F.Cu at (62.0, 92.0)
- added REF**: stencil-registration, myfootprints:stencil-registration, F.Cu at (128.0, 158.0)
- added REF**: stencil-registration, myfootprints:stencil-registration, F.Cu at (128.0, 92.0)
- added REF**: stencil-registration, myfootprints:stencil-registration, F.Cu at (62.0, 158.0)
- added REF**: OSHW-Logo2_9.8x8mm_SilkScreen, Symbol:OSHW-Logo2_9.8x8mm_SilkScreen, F.Cu at (85.1, 171.1)
- R18: value 0 -> 49.9; footprint Resistor_SMD:R_1210_3225Metric -> Resistor_SMD:R_0805_2012Metric
- R6: value 22k -> 20k
- U35: value STM32L072CBT6 -> STM32L151CCT6
- moved R18 24.9 mm to (78.9, 45.5), turned to 90 degrees
- moved C1 4.32 mm to (82.9, 43.9)
- moved R20 0.25 mm to (87.0, 125.8)
- moved C47 0.08 mm to (84.2, 128.2)
- moved C36 0.05 mm to (100.8, 138.9)
- turned C18 to 180 degrees
Connections:
- C23 pad 1: Net-(C23-Pad1) -> Net-(JP1-A)
- L3 pad 2: Net-(C23-Pad1) -> Net-(JP1-A)
- R1 pad 2: /Power/1V2_RUN -> Net-(JP2-B)
- R16 pad 1: Net-(C23-Pad1) -> Net-(JP1-A)
- R18 pad 1: Net-(C23-Pad1) -> Net-(U3-AVP)
- R18 pad 2: +5V -> GNDA
- TP1 pad 1: Net-(C23-Pad1) -> Net-(JP1-A)
- U19 pad 11: unconnected-(U19-?-Pad11) -> Net-(R46-Pad1)
- U20 pad 11: unconnected-(U20-?-Pad11) -> Net-(R44-Pad1)
- U25 pad 11: unconnected-(U25-?-Pad11) -> Net-(R47-Pad1)
- U26 pad 11: unconnected-(U26-?-Pad11) -> Net-(R45-Pad1)
- U3 pad 30: /Power/1V2_RUN -> Net-(JP2-B)
- U3 pad 4: unconnected-(U3-AVP-Pad4) -> Net-(U3-AVP)
- U35 pad 17: unconnected-(U35-PA7-Pad17) -> LDO_EN
- U4 pad 3: +3V3 -> LDO_EN
- U7 pad 3: +3V3 -> LDO_EN
Routing:
- net LDO_EN: track 0.00 -> 46.7 mm, vias 0 -> 2
- net Net-(JP1-A): track 0.00 -> 28.6 mm, vias 0 -> 2
- net Net-(C23-Pad1): track 28.3 -> 0.00 mm, vias 2 -> 0
- net /Power/1V2_RUN: track 19.6 -> 8.99 mm
- net Net-(JP2-B): track 0.00 -> 9.28 mm
- net GND: track 269.1 -> 276.5 mm, vias 251 -> 252
- net Net-(U3-AVP): track 0.00 -> 4.66 mm
- net +3V3: track 181.9 -> 177.3 mm
- net Net-(R44-Pad1): track 0.00 -> 2.97 mm, vias 0 -> 1
- net Net-(R45-Pad1): track 0.00 -> 2.26 mm, vias 0 -> 1
- net Net-(R47-Pad1): track 0.00 -> 2.22 mm, vias 0 -> 1
- net Net-(R46-Pad1): track 0.00 -> 2.05 mm, vias 0 -> 1
- net Net-(U3-ITH): track 4.85 -> 6.33 mm
- net +0V8: track 168.2 -> 167.0 mm
- net +5V: track 90.1 -> 90.9 mm
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
Commit message: updated L151 with L072 for qaxe+
Parts:
- U35: value STM32L151CCT6 -> STM32L072CBT6
Changed lines of the file:
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@@
 			)
 		)
-		(property "Value" "STM32L151CCT6"
+		(property "Value" "STM32L072CBT6"
 			(at 0 5.85 0)
 			(layer "F.Fab")
@@
 			)
 		)
-		(property "Manufacturer" "STM32L151CCT6"
+		(property "Manufacturer" "STM32L072CBT6"
 			(at 0 0 0)
 			(layer "F.Fab")
@@
 			)
 		)
-		(property "OrderNr" "497-19371-1-ND"
+		(property "OrderNr" "497-17503-ND"
 			(at 0 0 0)
 			(layer "F.Fab")
@@
 			(remove_unused_layers no)
 			(net 1 "GND")
-			(pinfunction "SGND")
+			(pinfunction "PGND")
 			(pintype "power_in")
 		)
@@
 			(remove_unused_layers no)
 			(net 1 "GND")
-			(pinfunction "SGND")
+			(pinfunction "PGND")
 			(pintype "power_in")
 		)
@@
 			(remove_unused_layers no)
 			(net 1 "GND")
-			(pinfunction "SGND")
+			(pinfunction "PGND")
 			(pintype "power_in")
 		)
@@
 			(remove_unused_layers no)
 			(net 1 "GND")
-			(pinfunction "SGND")
+			(pinfunction "PGND")
 			(pintype "power_in")
 		)
@@
 			(remove_unused_layers no)
 			(net 1 "GND")
-			(pinfunction "SGND")
+			(pinfunction "PGND")
 			(pintype "power_in")
 		)
@@
 			(layers "B.Cu")
 			(net 1 "GND")
-			(pinfunction "SGND")
+			(pinfunction "PGND")
 			(pintype "power_in")
 		)
@@
 			(layers "F.Cu" "F.Mask")
 			(net 1 "GND")
-			(pinfunction "SGND")
+			(pinfunction "PGND")
 			(pintype "power_in")
 		)
@@
 			(remove_unused_layers no)
 			(net 1 "GND")
-			(pinfunction "SGND")
+			(pinfunction "PGND")
 			(pintype "power_in")
 		)
@@
 			(remove_unused_layers no)
 			(net 1 "GND")
-			(pinfunction "SGND")
+			(pinfunction "PGND")
 			(pintype "power_in")
 		)
@@
 			(remove_unused_layers no)
 			(net 1 "GND")
-			(pinfunction "SGND")
+			(pinfunction "PGND")
 			(pintype "power_in")
 		)
@@
 			(remove_unused_layers no)
 			(net 1 "GND")
-			(pinfunction "SGND")
+			(pinfunction "PGND")
 			(pintype "power_in")
 		)
